File: ir_emitter.kicad_sch (KiCad schematic)
At the start: 35 parts, among them Q2 2N7002, Q3 2N7002, Q4 2N7002, Q5 2N7002, Q6 2N7002

Commit message: schematic: all errors and warnings gone
Parts:
- renumbered TP2 to TP3, TP3 to TP4, TP4 to TP5, TP5 to TP6, TP6 to TP7
Changed lines of the file:
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@@
 		(dnp no)
 		(fields_autoplaced yes)
-		(property "Reference" "TP2"
+		(property "Reference" "TP3"
 			(at 35.56 79.5019 0)
 			(effects
@@
 			(project ""
 				(path "/0ec4df52-ef34-4d49-9154-02bae5c96110/78e3f72c-305d-44d9-8e6b-dc611c685e57"
-					(reference "TP2")
+					(reference "TP3")
 					(unit 1)
 				)
@@
 		(dnp no)
 		(fields_autoplaced yes)
-		(property "Reference" "TP5"
+		(property "Reference" "TP6"
 			(at 187.96 88.3919 0)
 			(effects
@@
 			(project "RoboMaus"
 				(path "/0ec4df52-ef34-4d49-9154-02bae5c96110/78e3f72c-305d-44d9-8e6b-dc611c685e57"
-					(reference "TP5")
+					(reference "TP6")
 					(unit 1)
 				)
@@
 		(dnp no)
 		(fields_autoplaced yes)
-		(property "Reference" "TP3"
+		(property "Reference" "TP4"
 			(at 86.36 83.3119 0)
 			(effects
@@
 			(project "RoboMaus"
 				(path "/0ec4df52-ef34-4d49-9154-02bae5c96110/78e3f72c-305d-44d9-8e6b-dc611c685e57"
-					(reference "TP3")
+					(reference "TP4")
 					(unit 1)
 				)
@@
 		(dnp no)
 		(fields_autoplaced yes)
-		(property "Reference" "TP4"
+		(property "Reference" "TP5"
 			(at 137.16 85.8519 0)
 			(effects
@@
 			(project "RoboMaus"
 				(path "/0ec4df52-ef34-4d49-9154-02bae5c96110/78e3f72c-305d-44d9-8e6b-dc611c685e57"
-					(reference "TP4")
+					(reference "TP5")
 					(unit 1)
 				)
@@
 		(dnp no)
 		(fields_autoplaced yes)
-		(property "Reference" "TP6"
+		(property "Reference" "TP7"
 			(at 234.95 84.5819 0)
 			(effects
@@
 			(project "RoboMaus"
 				(path "/0ec4df52-ef34-4d49-9154-02bae5c96110/78e3f72c-305d-44d9-8e6b-dc611c685e57"
-					(reference "TP6")
-					(unit 1)
-				)
+					(reference "TP7")
+					(unit 1)
+				)

Commit message: pcb: all wired up, most warnings can't be fixed.
Parts:
- IRE1: renamed from TP3; value Emitter1 -> Testpoint
- IRE2: renamed from TP4; value Emitter2 -> Testpoint
- IRE3: renamed from TP5; value Emitter3 -> Testpoint
- IRE4: renamed from TP6; value Emitter4 -> Testpoint
- IRE5: renamed from TP7; value Emitter5 -> Testpoint
Changed lines of the file:
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@@
 		(dnp no)
 		(fields_autoplaced yes)
-		(property "Reference" "TP3"
+		(property "Reference" "IRE1"
 			(at 35.56 79.5019 0)
 			(effects
@@
 			)
 		)
-		(property "Value" "Emitter1"
+		(property "Value" "Testpoint"
 			(at 35.56 82.0419 0)
 			(effects
@@
 			(project ""
 				(path "/0ec4df52-ef34-4d49-9154-02bae5c96110/78e3f72c-305d-44d9-8e6b-dc611c685e57"
-					(reference "TP3")
+					(reference "IRE1")
 					(unit 1)
 				)
@@
 		(dnp no)
 		(fields_autoplaced yes)
-		(property "Reference" "TP6"
+		(property "Reference" "IRE4"
 			(at 187.96 88.3919 0)
 			(effects
@@
 			)
 		)
-		(property "Value" "Emitter4"
+		(property "Value" "Testpoint"
 			(at 187.96 90.9319 0)
 			(effects
@@
 			(project "RoboMaus"
 				(path "/0ec4df52-ef34-4d49-9154-02bae5c96110/78e3f72c-305d-44d9-8e6b-dc611c685e57"
-					(reference "TP6")
+					(reference "IRE4")
 					(unit 1)
 				)
@@
 		(dnp no)
 		(fields_autoplaced yes)
-		(property "Reference" "TP4"
+		(property "Reference" "IRE2"
 			(at 86.36 83.3119 0)
 			(effects
@@
 			)
 		)
-		(property "Value" "Emitter2"
+		(property "Value" "Testpoint"
 			(at 86.36 85.8519 0)
 			(effects
@@
 			(project "RoboMaus"
 				(path "/0ec4df52-ef34-4d49-9154-02bae5c96110/78e3f72c-305d-44d9-8e6b-dc611c685e57"
-					(reference "TP4")
+					(reference "IRE2")
 					(unit 1)
 				)
@@
 		(dnp no)
 		(fields_autoplaced yes)
-		(property "Reference" "TP5"
+		(property "Reference" "IRE3"
 			(at 137.16 85.8519 0)
 			(effects
@@
 			)
 		)
-		(property "Value" "Emitter3"
+		(property "Value" "Testpoint"
 			(at 137.16 88.3919 0)
 			(effects
@@
 			(project "RoboMaus"
 				(path "/0ec4df52-ef34-4d49-9154-02bae5c96110/78e3f72c-305d-44d9-8e6b-dc611c685e57"
-					(reference "TP5")
+					(reference "IRE3")
 					(unit 1)
 				)
@@
 		(dnp no)
 		(fields_autoplaced yes)
-		(property "Reference" "TP7"
+		(property "Reference" "IRE5"
 			(at 234.95 84.5819 0)
 			(effects
@@
 			)
 		)
-		(property "Value" "Emitter5"
+		(property "Value" "Testpoint"
 			(at 234.95 87.1219 0)
 			(effects
@@
 			(project "RoboMaus"
 				(path "/0ec4df52-ef34-4d49-9154-02bae5c96110/78e3f72c-305d-44d9-8e6b-dc611c685e57"
-					(reference "TP7")
-					(unit 1)
-				)
+					(reference "IRE5")
+					(unit 1)
+				)
